File: payload_hardware_design/adc.kicad_sch (KiCad schematic)
At the start: 0 parts

Commit message: making the PCB schematic
Parts:
- added C53, C54, C55, C56, C57, C58, C59: C, symbol Device:C
- added FB1: FerriteBead, symbol Device:FerriteBead
- added IC8: MCP3464RT-E_NC, QFN40P300X300X60-21N-D, symbol payload-sym:MCP3464RT-E_NC
- added R38, R65, R66, R67, R68, R69, R70, R71, R72, R73, R74, R75, R76, R77, R78: R_US, symbol Device:R_US
- added TP15: TestPoint, symbol Connector:TestPoint
- added U6: MCP1754ST-3302E/CB, SOT-23A_MC_MCH, symbol payload-sym:MCP1754ST-3302E_CB
Connections:
- new net: IC8.5 (CH2), R72.1
- new net: IC8.10 (CH7), R77.1
- new net: IC8.11 (~{CS}), R38.2
- new net: IC8.12 (SCK), R65.2
- new net: IC8.13 (SDI), R66.2
- new net: IC8.14 (SDO), R67.2
- new net: IC8.15 (~{IRQ}/MDAT), R68.2
- new net: IC8.16 (MCLK), R69.2
- new net: C58.1, C59.1, IC8.2 (REFIN+/OUT)
- new net: C56.2, IC8.20 (AGND), IC8.21 (EP)
- new net: IC8.3 (CH0), R70.1
- new net: IC8.4 (CH1), R71.1
- new net: IC8.6 (CH3), R73.1
- new net: IC8.7 (CH4), R74.1
- new net: IC8.8 (CH5), R75.1
- new net: IC8.9 (CH6), R76.1
- new net AGND: C57.2, C58.2, C59.2, IC8.1 (REFIN-), R77.2, R78.2
- new net GNDREF: C53.2, C54.2, C55.2, IC8.17 (DGND), R78.1, U6.1 (GND)
- new net SYS_5V: C53.1, U6.3 (VIN)
- new net VCC_3V3: C55.1, FB1.2, IC8.18 (DVDD)
- new net VDD_ADC: C54.1, C56.1, C57.1, FB1.1, IC8.19 (AVDD), TP15.1, U6.2 (VOUT)
Other:
- note added: "ADC"
- note added: "High PSRR LDO"
