File: payload_hardware_design/emmc.kicad_sch (KiCad schematic)
At the start: 1 part, among them U7 EMMC16G-TB29-PZ90

Commit message: making the PCB schematic
Parts:
- added C60, C61, C62, C63, C64, C65, C66, C67: C, symbol Device:C
- added R79, R80, R81, R82, R83, R84, R85, R86, R87, R88, R89, R90: R_US, symbol Device:R_US
Connections:
- net EMMC_DATA0: now reaches U7.A3 (DAT0)
- net EMMC_DATA0: now also R84.2
- net EMMC_DATA1: now reaches U7.A4 (DAT1)
- net EMMC_DATA1: now also R83.2
- net EMMC_DATA2: now reaches U7.A5 (DAT2)
- net EMMC_DATA2: now also R86.2
- net GNDREF: now reaches U7.A6 (VSS)
- net GNDREF: now also U7.C4 (VSSQ), U7.E7 (VSS), U7.G5 (VSS), U7.J5 (VSS), U7.K8 (VSS), U7.N2 (VSSQ), C60.2, C61.2, C62.2, C63.2, C64.2, C65.2, C66.2, C67.2, R80.2
- net EMMC_DATA3: now reaches U7.B2 (DAT3)
- net EMMC_DATA3: now also R85.2
- net EMMC_DATA4: now reaches U7.B3 (DAT4)
- net EMMC_DATA4: now also R88.2
- net EMMC_DATA5: now reaches U7.B4 (DAT5)
- net EMMC_DATA5: now also R87.2
- net EMMC_DATA6: now reaches U7.B5 (DAT6)
- net EMMC_DATA6: now also R90.2
- net EMMC_DATA7: now reaches U7.B6 (DAT7)
- net EMMC_DATA7: now also R89.2
- net at U7.C2 (VDDI): now also C67.1
- net VCC_1V8: now reaches U7.C6 (VCCQ)
- net VCC_1V8: now also U7.M4 (VCCQ), C64.1, C65.1, C66.1, R81.1, R82.1, R83.1, R84.1, R85.1, R86.1, R87.1, R88.1, R89.1, R90.1
- net VCC_3V3: now reaches U7.E6 (VCC)
- net VCC_3V3: now also U7.F5 (VCC), U7.K9 (VCC), C60.1, C61.1, C62.1, C63.1
- net EMMC_DS: now reaches U7.H5 (DS)
- net EMMC_DS: now also R80.1
- net EMMC_RSTn: now reaches U7.K5 (RST_n)
- net EMMC_RSTn: now also R82.2
- net EMMC_CMD: now reaches U7.M5 (CMD)
- net EMMC_CMD: now also R81.2
- net at U7.M6 (CLK): now also R79.2
- new net EMMC_CLK: R79.1
Other:
- note added: "EMMC"
- moved on the sheet: U7A, U7B
