File: hardware/soc_2.kicad_sch (KiCad schematic)
At the start: 1 part, among them U4 MPFS025T-FCVG484E

Commit message: update FPGA banks schematics
Changed lines of the file:
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@@
 	(symbol
 		(lib_id "payload-sym:MPFS025T-FCVG484E")
-		(at 24.13 16.51 0)
+		(at 33.02 38.1 0)
 		(unit 1)
 		(body_style 1)
@@
 		(dnp no)
 		(property "Reference" "U4"
-			(at 130.81 6.35 0)
+			(at 91.694 27.94 0)
 			(show_name no)
 			(do_not_autoplace no)
@@
 		)
 		(property "Value" "MPFS025T-FCVG484E"
-			(at 130.81 8.89 0)
+			(at 91.694 30.48 0)
 			(show_name no)
 			(do_not_autoplace no)
@@
 		)
 		(property "Footprint" "MPFS250T/MPFS160T/MPFS095T/MPFS025T-FCVG484_MCH"
-			(at 24.13 16.51 0)
+			(at 33.02 38.1 0)
 			(hide yes)
 			(show_name no)
@@
 		)
 		(property "Datasheet" "MPFS025T-FCVG484E"
-			(at 24.13 16.51 0)
+			(at 33.02 38.1 0)
 			(hide yes)
 			(show_name no)
@@
 		)
 		(property "Description" ""
-			(at 24.13 16.51 0)
+			(at 33.02 38.1 0)
 			(hide yes)
 			(show_name no)
@@
 		(fields_autoplaced yes)
 		(property "Reference" "U4"
-			(at 429.26 44.45 0)
+			(at 381.254 44.45 0)
 			(show_name no)
 			(do_not_autoplace no)
@@
 		)
 		(property "Value" "MPFS025T-FCVG484E"
-			(at 429.26 46.99 0)
+			(at 381.254 46.99 0)
 			(show_name no)
 			(do_not_autoplace no)
@@
 		(fields_autoplaced yes)
 		(property "Reference" "U4"
-			(at 133.35 152.4 0)
+			(at 85.344 152.4 0)
 			(show_name no)
 			(do_not_autoplace no)
@@
 		)
 		(property "Value" "MPFS025T-FCVG484E"
-			(at 133.35 154.94 0)
+			(at 85.344 154.94 0)
 			(show_name no)
 			(do_not_autoplace no)
