File: hardware/power_supply.kicad_sch (KiCad schematic)
At the start: 122 parts, among them IC1 MIC5504-2.5YM5-TR, IC2 TLV62569DBVT, IC3 MIC23303YML-TR, IC4 MIC23303YML-TR, IC5 MIC23303YML-TR, J1 Conn_01x02, Q1 RQ3E120ATTB, Q2 MMBT3906LT3G, Q3 RQ3E120ATTB, Q4 RQ3E120ATTB, Q5 BCM857BS-7-F, Q6 RQ3E120ATTB, Q7 BCM857BS-7-F, Q8 BCM857BS-7-F, Q9 BCM857BS-7-F, U1 ATL431AIDBZR, U2 MIC22950YML-TR, U3 MCP1725T-ADJE/MC

Commit message: updated schematic
Changed lines of the file:
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@@
 			(font
 				(size 3.81 3.81)
-				(thickness 1.016)
-				(bold yes)
+				(thickness 0.4763)
 			)
 		)
@@
 			(font
 				(size 3.81 3.81)
-				(thickness 1.016)
-				(bold yes)
+				(thickness 0.4763)
 			)
 		)
@@
 			(font
 				(size 3.81 3.81)
-				(thickness 1.016)
-				(bold yes)
+				(thickness 0.4763)
 			)
 		)
@@
 			(font
 				(size 3.81 3.81)
-				(thickness 1.016)
-				(bold yes)
+				(thickness 0.4763)
 			)
 		)
@@
 	(text "VIO_ENABLE"
 		(exclude_from_sim no)
-		(at 253.492 24.892 0)
+		(at 322.58 18.034 0)
 		(effects
 			(font
 				(size 3.81 3.81)
-				(thickness 1.016)
-				(bold yes)
+				(thickness 0.4763)
 			)
 		)
@@
 			(font
 				(size 3.81 3.81)
-				(thickness 1.016)
-				(bold yes)
+				(thickness 0.4763)
 			)
 		)
@@
 			(font
 				(size 3.81 3.81)
-				(thickness 1.016)
-				(bold yes)
+				(thickness 0.4763)
 			)
 		)
@@
 			(font
 				(size 3.81 3.81)
-				(thickness 1.016)
-				(bold yes)
+				(thickness 0.4763)
 			)
 		)
@@
 			(font
 				(size 3.81 3.81)
-				(thickness 1.016)
-				(bold yes)
+				(thickness 0.4763)
 			)
 		)
