File: hardware/communication.kicad_sch (KiCad schematic)
At the start: 20 parts, among them IC10 TCA9517DGKRQ1, IC9 TCA9517DGKRQ1, U8 SN65HVD234QDRQ1

Commit message: need finish io banks pinouts
Parts:
- added C181, C183: C, symbol Device:C
- added IC15: W25Q128JVSIQ, SOIC127P790X216-8N, symbol payload-sym:W25Q128JVSIQ
- added R121, R122, R123, R124, R125, R126, R127, R128, R129, R130, R131, R132, R133: R_US, symbol Device:R_US
- added TP17, TP18, TP19, TP20, TP21, TP22, TP23: TestPoint, symbol Connector:TestPoint
- added U16: MPFS025T-FCVG484E, MPFS250T/MPFS160T/MPFS095T/MPFS025T-FCVG484_MCH, symbol payload-sym:MPFS025T-FCVG484E
Connections:
- net GNDREF: now also C181.1, C183.1, IC15.4 (GND), R123.2, R126.2
- new net: R125.2, U16.F7 (SDO)
- new net: IC15.7 (/HOLD_OR_/RESET_(IO3)), R133.2
- new net: R121.1, U16.E8 (TDO)
- new net: R127.2, U16.G10 (FF_EXIT_N)
- new net: R124.2, U16.E6 (SCK)
- new net: IC15.2 (DO_(IO1)), R132.2
- new net: IC15.3 (/WP_(IO2)), R131.2
- new net JTAG_TCK: R126.1, U16.E9 (TCK)
- new net JTAG_TDI: U16.G9 (TDI)
- new net JTAG_TDO: R121.2
- new net JTAG_TMS: U16.F8 (TMS)
- new net JTAG_TRSTB: R123.1, U16.G8 (TRSTB)
- new net SPI_EN: TP18.1, U16.H11 (SPI_EN)
- new net SPI_MISO: R132.1, TP21.1, U16.H10 (SDI)
- new net SPI_MODE: R128.2, R129.2, TP19.1, U16.H9 (IO_CFG_INTF)
- new net SPI_MOSI: IC15.5 (DI_(IO0)), R125.1, TP20.1
- new net SPI_SCK: IC15.6 (CLK), R124.1, TP23.1
- new net SPI_SS: IC15.1 (/CS), R130.2, TP22.1, U16.G7 (SS)
- new net SYS_RSTN: C181.2, R122.2, TP17.1, U16.H7 (DEVRST_N)
- new net VCC_3V3: C183.2, IC15.8 (VCC), R122.1, R127.1, R128.1, R129.1, R130.1, R131.1, R133.1
Other:
- note added: "JTAG/SPI BANK"
- note added: "PROGRAMING THE SPI FLASH USING EXTERNAL MASTER"
- note added: "SPI FLASH"
- moved on the sheet: C89, C90, C91, C92, IC10, IC9, R100, R101, R102, R103, R104, R92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

Commit message: updated hardware
Other:
- moved on the sheet: C89, C90, C91, IC9, R92
