File: hardware/unused_banks.kicad_sch (KiCad schematic)
At the start: 1 part, among them U9 MPFS025T-FCVG484E

Commit message: updated schematic
Parts:
- added U16: MPFS025T-FCVG484E, MPFS250T/MPFS160T/MPFS095T/MPFS025T-FCVG484_MCH, symbol payload-sym:MPFS025T-FCVG484E

Commit message: need finish io banks pinouts
Parts:
- removed unit 9 of U16
Other:
- moved on the sheet: U16G
