File: hardware/interfaces.kicad_sch (KiCad schematic)
At the start: 2 parts, among them J3 SSQ-126-04-G-D, J4 SSQ-126-04-G-D

Commit message: updated hardware
Connections:
- net PAYLOAD_R0_ENABLE: now reaches J3.18 (H1_18)
- net POWER_ENABLE: now reaches J3.20 (H1_20)
- net GND: now reaches J3.29 (H1_29)
- net GND: now also J3.30 (H1_30), J3.31 (H1_31), J3.32 (H1_32), J4.29 (H2_29), J4.30 (H2_30), J4.31 (H2_31), J4.32 (H2_32)
Other:
- moved on the sheet: J3

Commit message: updated schematic
Parts:
- added C185: C, symbol Device:C
- added J5: FFC_HDGC_1x22_0.5K-DX-22PWB, FFC_HDGC_1x22_0.5K-DX-22PWB:Conn_FFC_HDGC_1x22_0.5K-DX-22PWB, symbol payload-sym:FFC_HDGC_1x22_0.5K-DX-22PWB
- added R136: R_US, symbol Device:R_US
Connections:
- new net: J5.17, R136.1
- new net CAM_D0_N: J5.2
- new net CAM_D0_P: J5.3
- new net CAM_D1_N: J5.5
- new net CAM_D1_P: J5.6
- new net CAM_D2_N: J5.8
- new net CAM_D2_P: J5.9
- new net CAM_D3_N: J5.11
- new net CAM_D3_P: J5.12
- new net CAM_D4_N: J5.14
- new net CAM_D4_P: J5.15
- new net CSI1_PDWN: R136.2
- new net GNDREF: C185.2, J5.1, J5.10, J5.13, J5.16, J5.19, J5.4, J5.7, J5.MP
- new net I2C_SCL: J5.20
- new net I2C_SDA: J5.21
- new net VCC_3V3: C185.1, J5.22
Other:
- note added: "MIPI CSI"
- moved on the sheet: J3, J4
