File: hardware/max2771.kicad_sch (KiCad schematic)
At the start: 3 parts, among them IC7 MAX2771ETI+

Commit message: need some I/O adjustments
Parts:
- added C70, C71, C72, C73, C74, C75, C76, C77, C78, C79, C80, C81, C82, C83, C84: C, symbol Device:C
- added R137, R138, R139, R140, R141, R91: R_US, symbol Device:R_US
- added TP24, TP25, TP26, TP27, TP28, TP29, TP30: TestPoint, symbol Connector:TestPoint
Connections:
- net CLK_OUT: now also C84.2; no longer IC7.4 (CLKOUT)
- net GNDREF: now also C70.2, C71.2, C72.2, C73.2, C74.2, C75.2, C77.2, C78.2, C79.2, C80.2, C81.2, C82.2
- net VCC_ADC: now also IC7.22 (VCCRF), C70.1, C71.1
- net at IC7.1 (CPOUT): now also C77.1, R141.1, TP26.1
- net Q1: now reaches IC7.10 (Q1)
- net Q1: now also TP30.1
- net Q0: now reaches IC7.11 (Q0)
- net Q0: now also TP29.1
- net I0: now reaches IC7.12 (I0)
- net I0: now also TP28.1
- net I1: now reaches IC7.13 (I1)
- net I1: now also TP27.1
- net LD_TO_HOST: now reaches IC7.17 (LD)
- net LD_TO_HOST: now also TP24.1
- net at IC7.18 (SHDN): now also R91.2
- net VCC_VCO: now reaches IC7.2 (VCCCP)
- net VCC_VCO: now also IC7.28 (VCCVCO), IC7.6 (VCCD), C74.1, C75.1, C79.1, C80.1, C81.1, C82.1
- net at IC7.23 (LNAOUT_LO): now also R139.2
- net at IC7.24 (LNAOUT_HI): now also R137.2
- net at IC7.25 (MIXIN_HI): now also R138.2
- net at IC7.26 (MIXIN_LO): now also R140.2
- net VCC_IF: now reaches IC7.27 (VCCIF)
- net VCC_IF: now also C72.1, C73.1
- net at IC7.3 (XTAL): now also C83.1
- net ANAINOUT: no longer names the net of IC7.16 (ANAINOUT)
- net ANAIPOUT: no longer names the net of IC7.15 (ANAIPOUT)
- new net: C76.1, R137.1, R139.1
- new net: C84.1, IC7.4 (CLKOUT)
- new net: C76.2, R138.1, R140.1
- new net: C78.1, R141.2
- new net CLKIN_REF: C83.2
- new net SHDN: R91.1, TP25.1
Other:
- note added: "PROGRAMING THE SPI FLASH USING EXTERNAL MASTER"
- moved on the sheet: C68, C69

Commit message: need review of MAX2771 connections, LDOs in general, names for the PC104 pins and his connection to other devices, include or exclude devices
Parts:
- added C169, C171, C254, C255, C256, C257, C258, C259, C260: C, symbol Device:C
- added IC16, IC17: MAX8510EXK29+T, SOT65P210X110-5N, symbol payload-sym:MAX8510EXK29+T
- added J6: Conn_Coaxial, symbol Connector:Conn_Coaxial
- added L6: L, symbol Device:L
- added R144, R145, R146, R147, R148, R149: R_US, symbol Device:R_US
Connections:
- net VCC_VCO is gone; now on net VCC_D: C74.1, C75.1, C79.1, C80.1, C81.1, C82.1, IC7.2 (VCCCP), IC7.28 (VCCVCO), IC7.6 (VCCD)
- net GNDREF: now also C169.2, C254.2, C255.2, C257.2, C258.2, C259.2, IC16.2 (GND), IC17.2 (GND), J6.1 (In), R145.1, R146.1
- net VCC_ADC: now also C256.1, C257.1, C258.1, IC17.4 (BP)
- net at IC7.19 (LNAIN_HI): now also R145.2, R147.2
- net at IC7.20 (LNAIN_LO): now also R146.2, R148.2
- net VCC_IF renamed VCC_D
- new net: C256.2, IC17.5 (OUT)
- new net: L6.2, R147.1, R148.1
- new net: C171.2, IC16.5 (OUT)
- new net: C260.1, J6.2 (Ext)
- new net: C259.1, L6.1, R149.2
- new net: IC16.3 (~{SHDN}), IC17.3 (~{SHDN}), R144.2
- new net: C260.2, R149.1
- new net VCC_CP: C171.1, C254.1, C255.1, IC16.4 (BP)
- new net VERIFICAR: C169.1, IC16.1 (IN), IC17.1 (IN), R144.1
Other:
- moved on the sheet: C68, C69, C70, C71, C72, C73, C74, C75, C76, C77, C78, C79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
